Commit message: 20211206

File: my_niryo_robot_description/urdf/ned/niryo_ned.urdf.xacro (robot description, xacro)
@@ -1,6 +1,9 @@
-<robot xmlns:xacro="http://www.ros.org/wiki/xacro" name="niryo_ned">
+<?xml version="1.0"?>
+<robot xmlns:xacro="http://www.ros.org/wiki/xacro">
+  <xacro:macro name="niryo_ned">
     <!-- Import Properties -->
     <xacro:include filename="$(find niryo_robot_description)/urdf/ned/niryo_ned_param.urdf.xacro"/>
     <!-- Links -->
+<!--
     <link name="world"/>
     <joint name="joint_world" type="fixed">
@@ -9,4 +12,5 @@
         <origin xyz="0 0 0" rpy="0 0 0"/>
     </joint>
+-->
     <link name="base_link">
         <inertial>
@@ -254,3 +258,4 @@
     <link name="tool_link">
     </link>
+  </xacro:macro>
 </robot>

File: my_niryo_robot_description/urdf/ned/niryo_ned_robot.urdf.xacro (robot description, xacro)
@@ -1,14 +1,89 @@
-<robot xmlns:xacro="http://www.ros.org/wiki/xacro" name="niryo_ned">
-    <xacro:include filename="$(find niryo_robot_description)/urdf/ned/niryo_ned_camera.urdf.xacro"/>
-    <!-- gazebo joint state publisher for all joints. Necessary to control mors -->
-    <gazebo>
-        <plugin name="passive_joint_state_publisher" filename="libgazebo_ros_joint_state_publisher.so">
-            <jointName>joint_1, joint_2, joint_3, joint_4, joint_5, joint_6,
-                joint_base_to_mors_1, joint_base_to_mors_2
-            </jointName>
-            <updateRate>50.0</updateRate>
-            <alwaysOn>true</alwaysOn>
-        </plugin>
-    </gazebo>
+<?xml version="1.0"?>
+<robot xmlns:xacro="http://wiki.ros.org/xacro" name="ur5_robot">
+  <!--
+    This is a convenience top-level xacro which loads the macro for the UR5e
+    which defines the default values for the various "parameters files"
+    parameters for a UR5e.
+    This file is only useful when loading a stand-alone, completely isolated
+    robot with only default values for all parameters such as the kinematics,
+    visual and physical parameters and joint limits.
+    This file is not intended to be integrated into a larger scene or other
+    composite xacro.
+    Instead, xacro:include 'inc/ur5e_macro.xacro' and override the defaults
+    for the arguments to that macro.
+    Refer to 'inc/ur_macro.xacro' for more information.
+  -->
+    <xacro:include filename="$(find my_niryo_robot_description)/urdf/ned/niryo_ned.transmission.xacro"/>
+  <xacro:include filename="$(find my_niryo_robot_description)/urdf/ned/niryo_ned.urdf.xacro"/>
+  <xacro:niryo_ned/>
+  <xacro:include filename="$(find my_niryo_robot_description)/urdf/ned/niryo_ned_gripper.urdf.xacro"/>
+  <xacro:niryo_ned_gripper/>
+  <material name="LightGrey">
+      <color rgba="0.7 0.7 0.7 1.0" />
+  </material>
+  <material name="blue">
+      <color rgba="0 0 0.8 1" />
+  </material>
+  <material name="red">
+      <color rgba="0.8 0 0 1" />
+  </material>
+  <xacro:macro name="cylinder_inertia" params="m r h">
+        <inertia  ixx="${m*(3*r*r+h*h)/12}" ixy = "0" ixz = "0"
+                    iyy="${m*(3*r*r+h*h)/12}" iyz = "0"
+                    izz="${m*r*r/2}" />
+  </xacro:macro>
+  <xacro:macro name="box_inertia" params="m x y z">
+          <inertia  ixx="${m*(y*y+z*z)/12}" ixy = "0" ixz = "0"
+                    iyy="${m*(x*x+z*z)/12}" iyz = "0"
+                    izz="${m*(x*x+z*z)/12}" />
+  </xacro:macro>
+  <xacro:macro name="sphere_inertia" params="m r">
+          <inertia  ixx="${2*m*r*r/5}" ixy = "0" ixz = "0"
+                    iyy="${2*m*r*r/5}" iyz = "0"
+                    izz="${2*m*r*r/5}" />
+  </xacro:macro>
+  <link name="world" />
+  <link name="baseplate_link">
+    <visual>
+      <origin xyz="0 0 0.0" />
+      <geometry>
+        <box size="1.1 0.7 0.03" />
+      </geometry>
+      <material name="LightGrey"/>
+    </visual>
+    <inertial>
+      <mass value="10"/>
+      <xacro:box_inertia m="10" x="1.1" y="0.7" z="0.03"/>
+    </inertial>
+  </link>
+  <joint name="baseplate_joint" type="fixed">
+    <origin xyz="0 0 0" />
+    <parent link="world" />
+    <child link="baseplate_link" />
+  </joint>
+  <link name="mountingplate_link">
+    <visual>
+      <origin xyz="0 0 0.0" />
+      <geometry>
+        <box size="0.3 0.3 0.012" />
+      </geometry>
+      <material name="red"/>
+    </visual>
+    <inertial>
+      <mass value="1"/>
+      <xacro:box_inertia m="1" x="0.3" y="0.3" z="0.012"/>
+    </inertial>
+  </link>
+  <joint name="mountingplate_joint" type="fixed">
+    <origin xyz="0.0 -0.20 0.021" />
+    <parent link="baseplate_link" />
+    <child link="mountingplate_link" />
+  </joint>
+  <!-- robot to mouting_plate. -->
+  <joint name="mountingplate_link" type="fixed">
+    <parent link="mountingplate_link" />
+    <child link="base_link" />
+    <origin xyz="0.0 0.0 0.01" rpy="0.0 0.0 ${pi/2}"/>
+  </joint>
     <!-- Joint from tool_link to base_gripper -->
     <joint name="joint_to_gripper" type="fixed">
@@ -17,141 +92,5 @@
         <origin
                 xyz="0 0 0.005"
-                rpy="0 ${PI/2} ${PI/2}"/>
+                rpy="0 ${pi/2} ${pi/2}"/>
     </joint>
-    <!-- Base Gripper -->
-    <link name="base_gripper_1">
-        <inertial>
-            <origin xyz="0.0028582 0.0022204 0.023772"
-                    rpy="0 0 0"/>
-            <mass value="0.001"/>
-            <inertia
-                    ixx="1E-06"
-                    ixy="0.0"
-                    ixz="0.0"
-                    iyy="1E-06"
-                    iyz="0.0"
-                    izz="1E-06"/>
-        </inertial>
-        <visual>
-            <origin xyz="0 0 0"
-                    rpy="0 0 0"/>
-            <geometry>
-                <mesh
-                        filename="package://niryo_robot_description/meshes/gripper_1/base_gripper_1.STL"/>
-            </geometry>
-        </visual>
-        <collision>
-            <origin xyz="0 0 0"
-                    rpy="0 0 0"/>
-            <geometry>
-                <mesh
-                        filename="package://niryo_robot_description/meshes/gripper_1/base_gripper_1.STL"/>
-            </geometry>
-        </collision>
-    </link>
-    <!-- Mors 1 -->
-    <link
-            name="mors_1">
-        <inertial>
-            <origin xyz="-0.0049739 0.0067393 -0.023929"
-                    rpy="0 0 0"/>
-            <mass value="0.0067248"/>
-            <inertia
-                    ixx="1.1778E-06"
-                    ixy="-2.1129E-08"
-                    ixz="1.0185E-07"
-                    iyy="1.3054E-06"
-                    iyz="1.7669E-07"
-                    izz="4.3534E-07"/>
-        </inertial>
-        <visual>
-            <origin xyz="0 0 0"
-                    rpy="0 0 0"/>
-            <geometry>
-                <mesh
-                        filename="package://niryo_robot_description/meshes/gripper_1/mors_1.STL"/>
-            </geometry>
-            <material name="">
-                <color rgba="0.49804 0.49804 0.49804 1"/>
-            </material>
-        </visual>
-        <collision>
-            <origin xyz="0 0 0"
-                    rpy="0 0 0"/>
-            <geometry>
-                <mesh
-                        filename="package://niryo_robot_description/meshes/gripper_1/mors_1.STL"/>
-            </geometry>
-        </collision>
-    </link>
-    <joint
-            name="joint_base_to_mors_1"
-            type="prismatic">
-        <origin xyz="0.01455 -0.0796 0.0096137"
-                rpy="1.5708 0 0"/>
-        <parent link="base_gripper_1"/>
-        <child link="mors_1"/>
-        <axis xyz="0 1 0"/>
-        <limit lower="-0.01"
-               upper="0.01"
-               effort="1"
-               velocity="5"/>
-    </joint>
-    <!-- Mors 2 -->
-    <link
-            name="mors_2">
-        <inertial>
-            <origin xyz="-0.0049739 -0.0067393 -0.023929"
-                    rpy="0 0 0"/>
-            <mass value="0.0067248"/>
-            <inertia
-                    ixx="1.1778E-06"
-                    ixy="2.1129E-08"
-                    ixz="1.0185E-07"
-                    iyy="1.3054E-06"
-                    iyz="-1.7669E-07"
-                    izz="4.3534E-07"/>
-        </inertial>
-        <visual>
-            <origin xyz="0 0 0"
-                    rpy="0 0 0"/>
-            <geometry>
-                <mesh
-                        filename="package://niryo_robot_description/meshes/gripper_1/mors_2.STL"/>
-            </geometry>
-        </visual>
-        <collision>
-            <origin xyz="0 0 0"
-                    rpy="0 0 0"/>
-            <geometry>
-                <mesh
-                        filename="package://niryo_robot_description/meshes/gripper_1/mors_2.STL"/>
-            </geometry>
-        </collision>
-    </link>
-    <joint name="joint_base_to_mors_2"
-           type="prismatic">
-        <origin xyz="0.01455 -0.0796 -0.011066"
-                rpy="1.5708 0 0"/>
-        <parent link="base_gripper_1"/>
-        <child link="mors_2"/>
-        <axis xyz="0 -1 0"/>
-        <limit lower="-0.01"
-               upper="0.01"
-               effort="1"
-               velocity="5"/>
-    </joint>
-    <!-- Transmissions -->
-    <xacro:SimpleTransmissionEffort n="7" joint="joint_base_to_mors_1"/>
-    <xacro:SimpleTransmissionEffort n="8" joint="joint_base_to_mors_2"/>
-    <!-- material -->
-    <gazebo reference="base_gripper_1">
-        <material>Gazebo/DarkGrey</material>
-    </gazebo>
-    <gazebo reference="mors_1">
-        <material>Gazebo/DarkGrey</material>
-    </gazebo>
-    <gazebo reference="mors_2">
-        <material>Gazebo/DarkGrey</material>
-    </gazebo>
 </robot>
