Commit message: 20211211

File: my_niryo_robot_description/urdf/ned/niryo_ned_robot.urdf.xacro (robot description, xacro)
@@ -60,27 +60,9 @@
     <child link="baseplate_link" />
   </joint>
-  <link name="mountingplate_link">
-    <visual>
-      <origin xyz="0 0 0.0" />
-      <geometry>
-        <box size="0.3 0.3 0.012" />
-      </geometry>
-      <material name="red"/>
-    </visual>
-    <inertial>
-      <mass value="1"/>
-      <xacro:box_inertia m="1" x="0.3" y="0.3" z="0.012"/>
-    </inertial>
-  </link>
-  <joint name="mountingplate_joint" type="fixed">
-    <origin xyz="0.0 -0.20 0.021" />
+  <!-- robot to baseplate_joint. -->
+  <joint name="mountingplate_link" type="fixed">
     <parent link="baseplate_link" />
-    <child link="mountingplate_link" />
-  </joint>
-  <!-- robot to mouting_plate. -->
-  <joint name="mountingplate_link" type="fixed">
-    <parent link="mountingplate_link" />
     <child link="base_link" />
-    <origin xyz="0.0 0.0 0.01" rpy="0.0 0.0 ${pi/2}"/>
+    <origin xyz="0.0 -0.20 0.021" rpy="0.0 0.0 ${pi/2}"/>
   </joint>
     <!-- Joint from tool_link to base_gripper -->

Commit message: 20220112

File: my_niryo_robot_description/urdf/ned/niryo_ned_robot.urdf.xacro (robot description, xacro)
@@ -54,13 +54,14 @@
   </link>
   <joint name="baseplate_joint" type="fixed">
-    <origin xyz="0 0 0" />
+    <origin xyz="0.20 0 0" rpy="0.0 0.0 ${pi/2}"/>
     <parent link="world" />
     <child link="baseplate_link" />
   </joint>
+world
   <!-- robot to baseplate_joint. -->
   <joint name="mountingplate_link" type="fixed">
-    <parent link="baseplate_link" />
+    <parent link="world" />
     <child link="base_link" />
-    <origin xyz="0.0 -0.20 0.021" rpy="0.0 0.0 ${pi/2}"/>
+    <origin xyz="0.0 0.0 0.021" rpy="0.0 0.0 0"/>
   </joint>
     <!-- Joint from tool_link to base_gripper -->

Commit message: 20220114

File: my_niryo_robot_description/urdf/ned/niryo_ned_robot.urdf.xacro (robot description, xacro)
@@ -77,3 +77,10 @@
     </joint>
   -->
+  <!-- tool center point -->
+  <link name="tcp_link" />
+  <joint name="tool0_link" type="fixed">
+    <parent link="tool_link" />
+    <child link="tcp_link" />
+    <origin xyz="0.0 0.0 0.0" rpy="0.0 0.0 0.0"/>
+  </joint>
 </robot>
