Commit message: 20230614

File: my_niryo_robot_description/urdf/ned/niryo_ned_gripper.urdf.xacro (robot description, xacro)
@@ -33,4 +33,7 @@
                         filename="package://niryo_robot_description/meshes/gripper_1/base_gripper_1.STL"/>
             </geometry>
+            <material name="">
+                <color rgba="0.49804 0.49804 0.49804 1"/>
+            </material>
         </visual>
         <collision>
@@ -113,4 +116,7 @@
                         filename="package://niryo_robot_description/meshes/gripper_1/mors_2.STL"/>
             </geometry>
+            <material name="">
+                <color rgba="0.49804 0.49804 0.49804 1"/>
+            </material>
         </visual>
         <collision>
